Commit message: Add MOMA

File: urdf/tm12.urdf (robot description, URDF)
Before this commit: robot tm12, 9 links, 8 joints
Links:
- link link_0: geometry collision mesh filename=package://gazebo_test_bed/meshes/tm12/collision/tm12-base_c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; visual mesh filename=package://gazebo_test_bed/meshes/tm12/visual/tm12-base.obj
- link link_1: geometry collision mesh filename=package://gazebo_test_bed/meshes/tm12/collision/tmr_750w_01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; visual mesh filename=package://gazebo_test_bed/meshes/tm12/visual/tmr_750w_01.obj
- link link_2: geometry collision mesh filename=package://gazebo_test_bed/meshes/tm12/collision/tm12-arm1_c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; visual mesh filename=package://gazebo_test_bed/meshes/tm12/visual/tm12-arm1.obj
- link link_3: geometry collision mesh filename=package://gazebo_test_bed/meshes/tm12/collision/tm12-arm2_c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; visual mesh filename=package://gazebo_test_bed/meshes/tm12/visual/tm12-arm2.obj
- link link_4: geometry collision mesh filename=package://gazebo_test_bed/meshes/tm5-900/collision/tmr_100w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; visual mesh filename=package://gazebo_test_bed/meshes/tm5-900/visual/tmr_100w_01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
- link link_5: geometry collision mesh filename=package://gazebo_test_bed/meshes/tm5-900/collision/tmr_100w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; visual mesh filename=package://gazebo_test_bed/meshes/tm5-900/visual/tmr_100w_02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
- link link_6: geometry collision mesh filename=package://gazebo_test_bed/meshes/tm5-900/collision/tmr_ee_c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; visual mesh filename=package://gazebo_test_bed/meshes/tm5-900/visual/tmr_ee.obj

File: xacro/macro.gazebo.xacro (robot description, xacro)
@@ -1,24 +1,16 @@
 <?xml version="1.0"?>
 <robot xmlns:xacro="http://www.ros.org/wiki/xacro">
-  <xacro:macro name="tmr_gazebo" params="ns prefix">
-    <gazebo reference="${prefix}link_1">
-      <selfCollide>true</selfCollide>
-    </gazebo>
-    <gazebo reference="${prefix}link_2">
-      <selfCollide>true</selfCollide>
-    </gazebo>
-    <gazebo reference="${prefix}link_3">
-      <selfCollide>true</selfCollide>
-    </gazebo>
-    <gazebo reference="${prefix}link_4">
-      <selfCollide>true</selfCollide>
-    </gazebo>
-    <gazebo reference="${prefix}link_5">
-      <selfCollide>true</selfCollide>
-    </gazebo>
-    <gazebo reference="${prefix}link_6">
-      <selfCollide>true</selfCollide>
-    </gazebo>
-    <!-- Gripper Gazebo 설정 추가 -->
+  <!--
+    tm12 고정 로봇 전용 gazebo 매크로.
+    mobile_manipulator 는 별도 파일에서 직접 ign_ros2_control 플러그인을 정의하므로
+    이 매크로를 호출하지 않음.
+  -->
+  <xacro:macro name="tmr_gazebo" params="ns prefix robot_namespace:=''">
+    <gazebo reference="${prefix}link_1"><selfCollide>true</selfCollide></gazebo>
+    <gazebo reference="${prefix}link_2"><selfCollide>true</selfCollide></gazebo>
+    <gazebo reference="${prefix}link_3"><selfCollide>true</selfCollide></gazebo>
+    <gazebo reference="${prefix}link_4"><selfCollide>true</selfCollide></gazebo>
+    <gazebo reference="${prefix}link_5"><selfCollide>true</selfCollide></gazebo>
+    <gazebo reference="${prefix}link_6"><selfCollide>true</selfCollide></gazebo>
     <gazebo reference="${prefix}gripper_link">
       <selfCollide>true</selfCollide>
@@ -27,8 +19,34 @@
       <mu2>0.9</mu2>
     </gazebo>
+    <gazebo reference="${prefix}gripper_surface_link">
+      <selfCollide>true</selfCollide>
+      <sensor name="gripper_contact_sensor" type="contact">
+        <contact>
+          <collision>${prefix}gripper_surface_link_collision</collision>
+        </contact>
+        <update_rate>30</update_rate>
+        <always_on>true</always_on>
+        <plugin filename="libignition-gazebo-contact-system.so"
+                name="ignition::gazebo::systems::Contact">
+        </plugin>
+      </sensor>
+    </gazebo>
+    <!-- ign_ros2_control 플러그인 → /controller_manager (tm12 전용) -->
     <gazebo>
       <plugin filename="ign_ros2_control-system"
               name="ign_ros2_control::IgnitionROS2ControlPlugin">
-        <parameters>$(find tm12_gazebo_moveit)/tm_config/ros2_controllers.yaml</parameters>
+        <parameters>$(find gazebo_test_bed)/tm_config/ros2_controllers.yaml</parameters>
+      </plugin>
+    </gazebo>
+    <!-- Dynamic Gripper Plugin -->
+    <gazebo>
+      <plugin filename="tm12_gazebo_moveit/libdynamic_gripper_plugin.so"
+              name="dynamic_gripper::DynamicGripperPlugin">
+        <parent_link>${prefix}gripper_surface_link</parent_link>
+        <contact_sensor_topic>/world/empty/model/tm12/link/gripper_surface_link/sensor/gripper_contact_sensor/contact</contact_sensor_topic>
+        <attach_topic>/tm12_gripper/attach</attach_topic>
+        <detach_topic>/tm12_gripper/detach</detach_topic>
+        <state_topic>/tm12_gripper/state</state_topic>
+        <attach_distance>0.01</attach_distance>
       </plugin>
     </gazebo>

File: xacro/macro.tm12.urdf.xacro (robot description, xacro)
@@ -1,6 +1,6 @@
 <?xml version="1.0"?>
 <robot xmlns:xacro="http://www.ros.org/wiki/xacro">
-  <xacro:include filename="$(find tm12_gazebo_moveit)/xacro/macro.inertial.xacro" />
-  <xacro:macro name="tm12" params="ns prefix color:=orange format:=obj
+  <xacro:include filename="$(find gazebo_test_bed)/xacro/macro.inertial.xacro" />
+  <xacro:macro name="tm12" params="ns prefix color:=grey format:=obj
     joint_1_lower_limit:=${radians(-330)}    joint_1_upper_limit:=${radians(330)}
     joint_2_lower_limit:=${radians(-180)}    joint_2_upper_limit:=${radians(180)}
@@ -23,19 +23,18 @@
     safety_limits:=false safety_pos_margin:=0.15
     safety_k_position:=20">
-   <xacro:property name="damping_factor" value="0.000"/>
-   <xacro:property name="d1" value="${damping_factor*0.1}"/>
-   <xacro:property name="d2" value="${damping_factor*0.1}"/>
-   <xacro:property name="d3" value="${damping_factor*0.1}"/>
-   <xacro:property name="d4" value="${damping_factor*0.1}"/>
-   <xacro:property name="d5" value="${damping_factor*0.1}"/>
-   <xacro:property name="d6" value="${damping_factor*0.1}"/>
-   <xacro:property name="friction_factor" value="0.000"/>
-   <xacro:property name="f1" value="${friction_factor*0.1}"/>
-   <xacro:property name="f2" value="${friction_factor*0.1}"/>
-   <xacro:property name="f3" value="${friction_factor*0.1}"/>
-   <xacro:property name="f4" value="${friction_factor*0.1}"/>
-   <xacro:property name="f5" value="${friction_factor*0.1}"/>
-   <xacro:property name="f6" value="${friction_factor*0.1}"/>
-    <!-- Inertia parameters -->
+    <xacro:property name="damping_factor" value="1000.0"/>
+    <xacro:property name="friction_factor" value="50.0"/>
+    <xacro:property name="d1" value="${damping_factor*0.1}"/>
+    <xacro:property name="d2" value="${damping_factor*0.1}"/>
+    <xacro:property name="d3" value="${damping_factor*0.1}"/>
+    <xacro:property name="d4" value="${damping_factor*0.1}"/>
+    <xacro:property name="d5" value="${damping_factor*0.1}"/>
+    <xacro:property name="d6" value="${damping_factor*0.1}"/>
+    <xacro:property name="f1" value="${friction_factor*0.1}"/>
+    <xacro:property name="f2" value="${friction_factor*0.1}"/>
+    <xacro:property name="f3" value="${friction_factor*0.1}"/>
+    <xacro:property name="f4" value="${friction_factor*0.1}"/>
+    <xacro:property name="f5" value="${friction_factor*0.1}"/>
+    <xacro:property name="f6" value="${friction_factor*0.1}"/>
     <xacro:property name="mass_0" value="1.0" />
     <xacro:property name="mass_1" value="7.6" />
@@ -65,18 +64,16 @@
     <xacro:property name="izz_5" value="${2643.21*unit_factor}" />
     <xacro:property name="izz_6" value="${1559.496*unit_factor}" />
-<!--LinkDescription-->
   <link name="${prefix}link_0">
     <visual>
       <geometry>
-        <mesh filename="package://tm12_gazebo_moveit/meshes/tm12/visual/tm12-base.${format}" />
-      </geometry>
-      <material name="${color}" />
-    </visual>
-    <collision>
-      <geometry>
-        <mesh filename="package://tm12_gazebo_moveit/meshes/tm12/collision/tm12-base_c.stl" />
-      </geometry>
-    </collision>
-<!--inertial-->
+        <mesh filename="package://gazebo_test_bed/meshes/tm12/visual/tm12-base.${format}" />
+      </geometry>
+      <material name="${color}" />
+    </visual>
+    <collision>
+      <geometry>
+        <mesh filename="package://gazebo_test_bed/meshes/tm12/collision/tm12-base_c.stl" />
+      </geometry>
+    </collision>
     <xacro:cylinder_inertial_z radius="0.06" length="0.05" mass="${mass_0}">
       <origin rpy="0.000000 0.000000 0.000000" xyz="0.000000 0.000000 0.000000" />
@@ -88,5 +85,4 @@
     <origin rpy="0.000000 -0.000000 0.000000" xyz="0.000000 0.000000 0.165200" />
     <axis xyz="0 0 1" />
-<!--limit-->
     <limit lower="${joint_1_lower_limit}" upper="${joint_1_upper_limit}" velocity="${joint_1_velocity_limit}" effort="${joint_1_effort_limit}" />
     <xacro:if value="${safety_limits}">
@@ -98,11 +94,11 @@
     <visual>
       <geometry>
-        <mesh filename="package://tm12_gazebo_moveit/meshes/tm12/visual/tmr_750w_01.${format}" />
-      </geometry>
-      <material name="${color}" />
-    </visual>
-    <collision>
-      <geometry>
-        <mesh filename="package://tm12_gazebo_moveit/meshes/tm12/collision/tmr_750w_01_c.stl" />
+        <mesh filename="package://gazebo_test_bed/meshes/tm12/visual/tmr_750w_01.${format}" />
+      </geometry>
+      <material name="${color}" />
+    </visual>
+    <collision>
+      <geometry>
+        <mesh filename="package://gazebo_test_bed/meshes/tm12/collision/tmr_750w_01_c.stl" />
       </geometry>
     </collision>
@@ -118,5 +114,4 @@
     <origin rpy="-1.570796 -1.570796 0.000000" xyz="0.000000 0.000000 0.000000" />
     <axis xyz="0 0 1" />
-<!--limit-->
     <limit lower="${joint_2_lower_limit}" upper="${joint_2_upper_limit}" velocity="${joint_2_velocity_limit}" effort="${joint_2_effort_limit}" />
     <xacro:if value="${safety_limits}">
@@ -128,11 +123,11 @@
     <visual>
       <geometry>
-        <mesh filename="package://tm12_gazebo_moveit/meshes/tm12/visual/tm12-arm1.${format}" />
-      </geometry>
-      <material name="${color}" />
-    </visual>
-    <collision>
-      <geometry>
-        <mesh filename="package://tm12_gazebo_moveit/meshes/tm12/collision/tm12-arm1_c.stl" />
+        <mesh filename="package://gazebo_test_bed/meshes/tm12/visual/tm12-arm1.${format}" />
+      </geometry>
+      <material name="${color}" />
+    </visual>
+    <collision>
+      <geometry>
+        <mesh filename="package://gazebo_test_bed/meshes/tm12/collision/tm12-arm1_c.stl" />
       </geometry>
     </collision>
@@ -148,5 +143,4 @@
     <origin rpy="0.000000 -0.000000 0.000000" xyz="0.636100 0.000000 0.000000" />
     <axis xyz="0 0 1" />
-<!--limit-->
     <limit lower="${joint_3_lower_limit}" upper="${joint_3_upper_limit}" velocity="${joint_3_velocity_limit}" effort="${joint_3_effort_limit}" />
     <xacro:if value="${safety_limits}">
@@ -158,11 +152,11 @@
     <visual>
       <geometry>
-        <mesh filename="package://tm12_gazebo_moveit/meshes/tm12/visual/tm12-arm2.${format}" />
-      </geometry>
-      <material name="${color}" />
-    </visual>
-    <collision>
-      <geometry>
-        <mesh filename="package://tm12_gazebo_moveit/meshes/tm12/collision/tm12-arm2_c.stl" />
+        <mesh filename="package://gazebo_test_bed/meshes/tm12/visual/tm12-arm2.${format}" />
+      </geometry>
+      <material name="${color}" />
+    </visual>
+    <collision>
+      <geometry>
+        <mesh filename="package://gazebo_test_bed/meshes/tm12/collision/tm12-arm2_c.stl" />
       </geometry>
     </collision>
@@ -178,5 +172,4 @@
     <origin rpy="0.000000 -0.000000 1.570796" xyz="0.557900 0.000000 -0.156300" />
     <axis xyz="0 0 1" />
-<!--limit-->
     <limit lower="${joint_4_lower_limit}" upper="${joint_4_upper_limit}" velocity="${joint_4_velocity_limit}" effort="${joint_4_effort_limit}" />
     <xacro:if value="${safety_limits}">
@@ -188,11 +181,11 @@
     <visual>
       <geometry>
-        <mesh filename="package://tm12_gazebo_moveit/meshes/tm5-900/visual/tmr_100w_01.${format}" />
-      </geometry>
-      <material name="${color}" />
-    </visual>
-    <collision>
-      <geometry>
-        <mesh filename="package://tm12_gazebo_moveit/meshes/tm5-900/collision/tmr_100w_01_c.stl" />
+        <mesh filename="package://gazebo_test_bed/meshes/tm5-900/visual/tmr_100w_01.${format}" />
+      </geometry>
+      <material name="${color}" />
+    </visual>
+    <collision>
+      <geometry>
+        <mesh filename="package://gazebo_test_bed/meshes/tm5-900/collision/tmr_100w_01_c.stl" />
       </geometry>
     </collision>
@@ -208,5 +201,4 @@
     <origin rpy="1.570796 -0.000000 0.000000" xyz="0.000000 -0.106000 0.000000" />
     <axis xyz="0 0 1" />
-<!--limit-->
     <limit lower="${joint_5_lower_limit}" upper="${joint_5_upper_limit}" velocity="${joint_5_velocity_limit}" effort="${joint_5_effort_limit}" />
     <xacro:if value="${safety_limits}">
@@ -218,11 +210,11 @@
     <visual>
       <geometry>
-        <mesh filename="package://tm12_gazebo_moveit/meshes/tm5-900/visual/tmr_100w_02.${format}" />
-      </geometry>
-      <material name="${color}" />
-    </visual>
-    <collision>
-      <geometry>
-        <mesh filename="package://tm12_gazebo_moveit/meshes/tm5-900/collision/tmr_100w_02_c.stl" />
+        <mesh filename="package://gazebo_test_bed/meshes/tm5-900/visual/tmr_100w_02.${format}" />
+      </geometry>
+      <material name="${color}" />
+    </visual>
+    <collision>
+      <geometry>
+        <mesh filename="package://gazebo_test_bed/meshes/tm5-900/collision/tmr_100w_02_c.stl" />
       </geometry>
     </collision>
@@ -238,5 +230,4 @@
     <origin rpy="1.570796 -0.000000 0.000000" xyz="0.000000 -0.113150 0.000000" />
     <axis xyz="0 0 1" />
-<!--limit-->
     <limit lower="${joint_6_lower_limit}" upper="${joint_6_upper_limit}" velocity="${joint_6_velocity_limit}" effort="${joint_6_effort_limit}" />
     <xacro:if value="${safety_limits}">
@@ -248,11 +239,11 @@
     <visual>
       <geometry>
-        <mesh filename="package://tm12_gazebo_moveit/meshes/tm5-900/visual/tmr_ee.${format}" />
-      </geometry>
-      <material name="${color}" />
-    </visual>
-    <collision>
-      <geometry>
-        <mesh filename="package://tm12_gazebo_moveit/meshes/tm5-900/collision/tmr_ee_c.stl" />
+        <mesh filename="package://gazebo_test_bed/meshes/tm5-900/visual/tmr_ee.${format}" />
+      </geometry>
+      <material name="${color}" />
+    </visual>
+    <collision>
+      <geometry>
+        <mesh filename="package://gazebo_test_bed/meshes/tm5-900/collision/tmr_ee_c.stl" />
       </geometry>
     </collision>
@@ -267,20 +258,18 @@
       <origin xyz="0 0 0" rpy="0 0 0"/>
       <geometry>
-        <mesh filename="package://tm12_gazebo_moveit/meshes/tm12/visual/gripper.stl" scale="1 1 1"/>
-      </geometry>
-      <material name="orange" />
+        <mesh filename="package://gazebo_test_bed/meshes/tm12/visual/gripper.stl" scale="1 1 1"/>
+      </geometry>
+      <material name="grey" />
     </visual>
     <collision>
       <origin xyz="0 0 0" rpy="0 0 0"/>
       <geometry>
-        <mesh filename="package://tm12_gazebo_moveit/meshes/tm12/visual/gripper.stl" scale="0.001 0.001 0.001"/>
-      </geometry>
-    </collision>
-    <inertial>
-      <origin xyz="0 0 0.05" rpy="0 0 0"/>
+        <mesh filename="package://gazebo_test_bed/meshes/tm12/visual/gripper.stl" scale="1 1 1"/>
+      </geometry>
+    </collision>
+    <inertial>
+      <origin xyz="0 0 0" rpy="0 0 0"/>
       <mass value="${mass_gripper}"/>
-      <inertia ixx="0.001" ixy="0.0" ixz="0.0"
-               iyy="0.001" iyz="0.0"
-               izz="0.001"/>
+      <inertia ixx="0.01" ixy="0.0" ixz="0.0" iyy="0.01" iyz="0.0" izz="0.01"/>
     </inertial>
   </link>
@@ -289,7 +278,45 @@
     <child link="${prefix}gripper_link"/>
     <origin xyz="0 0 0.0" rpy="3.14159 0 0"/>
-    <!-- 필요시 위치 조정: xyz="0 0 0.1" 등 -->
-  </joint>
-  <!-- ========================================== -->
+  </joint>
+  <gazebo reference="${prefix}gripper_joint">
+    <preserveFixedJoint>true</preserveFixedJoint>
+  </gazebo>
+  <link name="${prefix}gripper_surface_link">
+    <visual>
+      <origin xyz="0 0 0" rpy="0 0 0"/>
+      <geometry>
+        <sphere radius="0.01"/>
+      </geometry>
+      <material name="none">
+        <color rgba="1 0 0 0"/>
+      </material>
+    </visual>
+    <collision name="${prefix}gripper_surface_link">
+      <geometry>
+        <box size="0.01 0.01 0.01"/> </geometry>
+    </collision>
+    <inertial>
+      <mass value="0.01" />
+      <origin xyz="0 0 0" rpy="0 0 0" />
+      <inertia ixx="0.000001" ixy="0" ixz="0" iyy="0.000001" iyz="0" izz="0.000001" />
+    </inertial>
+    <sensor name="gripper_contact_sensor" type="contact">
+      <contact>
+        <collision>${prefix}gripper_surface_link</collision>
+      </contact>
+      <update_rate>30</update_rate>
+      <plugin filename="libignition-gazebo-contact-system" name="ignition::gazebo::systems::Contact">
+        <always_on>true</always_on>
+      </plugin>
+    </sensor>
+  </link>
+  <joint name="${prefix}gripper_surface_joint" type="fixed">
+    <parent link="${prefix}gripper_link"/>
+    <child link="${prefix}gripper_surface_link"/>
+    <origin xyz="0 0 -0.166" rpy="0 0 0"/>
+  </joint>
+  <gazebo reference="${prefix}gripper_surface_joint">
+    <preserveFixedJoint>true</preserveFixedJoint>
+  </gazebo>
   <link name="${prefix}base" />
   <joint name="${prefix}base_fixed_joint" type="fixed">
@@ -304,5 +331,4 @@
     <origin rpy="0.000000 0.000000 0.000000" xyz="0.000000 0.000000 0.000000" />
   </joint>
-<!--LinkDescription-->
-  </xacro:macro>
+</xacro:macro>
 </robot>

File: xacro/tm12.urdf.xacro (robot description, xacro)
@@ -5,8 +5,8 @@
   <xacro:arg name="color" default="none" />
   <xacro:arg name="trans_hw_iface" default="hardware_interface/PositionJointInterface" />
-  <xacro:include filename="$(find tm12_gazebo_moveit)/xacro/macro.gazebo.xacro" />
-  <xacro:include filename="$(find tm12_gazebo_moveit)/xacro/macro.transmission.xacro" />
-  <xacro:include filename="$(find tm12_gazebo_moveit)/xacro/macro.materials.xacro" />
-  <xacro:include filename="$(find tm12_gazebo_moveit)/xacro/macro.tm12.urdf.xacro" />
+  <xacro:include filename="$(find gazebo_test_bed)/xacro/macro.gazebo.xacro" />
+  <xacro:include filename="$(find gazebo_test_bed)/xacro/macro.transmission.xacro" />
+  <xacro:include filename="$(find gazebo_test_bed)/xacro/macro.materials.xacro" />
+  <xacro:include filename="$(find gazebo_test_bed)/xacro/macro.tm12.urdf.xacro" />
   <link name="world">
     <visual>
@@ -36,8 +36,43 @@
     <static>true</static>
   </gazebo>
+  <link name="support_block">
+    <visual>
+      <origin xyz="0 0 0" rpy="0 0 0"/>
+      <geometry>
+        <box size="0.2 0.2 0.63"/>
+      </geometry>
+      <material name="BlockGrey">
+        <color rgba="0.3 0.3 0.3 1.0"/>
+      </material>
+    </visual>
+    <collision>
+      <origin xyz="0 0 0" rpy="0 0 0"/>
+      <geometry>
+        <box size="0.2 0.2 0.63"/>
+      </geometry>
+    </collision>
+    <inertial>
+      <mass value="500.0"/>
+      <origin xyz="0 0 0" rpy="0 0 0"/>
+      <inertia ixx="16.58" ixy="0.0" ixz="0.0"
+               iyy="16.58" iyz="0.0"
+               izz="10.42"/>
+    </inertial>
+  </link>
+  <!-- Gazebo properties for support block -->
+  <gazebo reference="support_block">
+    <static>true</static>
+    <material>Gazebo/DarkGrey</material>
+  </gazebo>
+  <!-- Joint to attach support block to world -->
+  <joint name="world_to_support_block" type="fixed">
+    <parent link="world"/>
+    <child link="support_block"/>
+    <origin xyz="0.8 4.6 0.315" rpy="0.0 0.0 3.14159"/>
+  </joint>
   <joint name="world_to_base_fixed" type="fixed">
     <parent link="world"/>
     <child link="$(arg prefix)base"/>
-    <origin xyz="0.0 0.0 0.0" rpy="0.0 0.0 0.0"/>
+    <origin xyz="0.8 4.6 0.63" rpy="0.0 0.0 3.14159"/>
   </joint>
   <xacro:tmr_gazebo ns="$(arg ns)" prefix="$(arg prefix)" />
